File: hw/sch_pcb/TFI2CEXT01A.kicad_pcb (KiCad board)
At the start: 2 copper layers, 37.5 x 19 mm, 23 parts, among them J1 HEADER_1x03, J2 SM04B-GHS-TB, J3 SM04B-GHS-TB, M2 M3, U1 PCF8583, U2 74HC1G14GW, U3 MIC5504-3.3YM5

Commit message: The first layout
Parts:
- removed C5, C6: 100nF, Mlab_R:SMD-0603
- removed G***: LOGO, MLAB_LOGA:TF
- removed JP1, JP2: SolderJumper_3_Bridged12, Jumper:SolderJumper-3_P1.3mm_Bridged12_RoundedPad1.0x1.5mm
- removed M2: M3, Mlab_Mechanical:MountingHole_3mm
- removed R10: 10k, Mlab_R:SMD-0603
- removed U3: MIC5504-3.3YM5, Package_TO_SOT_SMD:SOT-23-5
- added D3: LED RED, Mlab_D:LED_1206, B.Cu at (15.0, -2.00)
- added J4: SM04B-GHS-TB, Connector_JST:JST_GH_SM04B-GHS-TB_1x04-1MP_P1.25mm_Horizontal, F.Cu at (33.2, -6.00)
- added M1: M3, Mlab_Mechanical:MountingHole_3mm, F.Cu at (31.5, -75.2)
- added R5: 10k, Mlab_R:SMD-0603, B.Cu at (49.6, -43.5)
- added R6: 10k, Mlab_R:SMD-0603, B.Cu at (46.2, -50.4)
- C1: value 1uF -> 10uF; footprint Mlab_R:SMD-0603 -> Mlab_R:SMD-0805
- C2: value 10uF -> 100nF; footprint Mlab_R:SMD-0805 -> Mlab_R:SMD-0603
- C3: value 10uF -> 1uF; footprint Mlab_R:SMD-0805 -> Mlab_R:SMD-0603
- D1: value ZENER-5.6V -> LED GREEN; footprint Mlab_D:Diode-MiniMELF_Standard -> Mlab_D:LED_1206
- D2: value LED RED -> BZX585-B5V6.115; footprint Mlab_D:LED_1206 -> Diode_SMD:D_SOD-523
- J1: value HEADER_1x03 -> SM04B-GHS-TB; footprint Connector_PinHeader_2.54mm:PinHeader_1x03_P2.54mm_Horizontal -> Connector_JST:JST_GH_SM04B-GHS-TB_1x04-1MP_P1.25mm_Horizontal
- J2: moved to F.Cu
- R1: value 470R -> 180R; footprint Mlab_R:SMD-0805 -> Mlab_R:SMD-0603
- R2: value 100R -> 10k; footprint Mlab_R:SMD-0805 -> Mlab_R:SMD-0603
- U1: value PCF8583 -> MIC5504-3.3YM5; footprint Mlab_IO:SOT176-1 -> Package_TO_SOT_SMD:SOT-23-5
- U2: value 74HC1G14GW -> TCA4307; footprint Package_TO_SOT_SMD:SOT-353_SC-70-5 -> Package_SO:VSSOP-8_3.0x3.0mm_P0.65mm
- moved R3 203.1 mm to (35.4, -56.4), turned to 0 degrees
- moved J1 195.5 mm to (2.80, -6.00), turned to 90 degrees
- moved R2 194.6 mm to (48.4, -46.4), turned to 0 degrees
- moved D2 194.0 mm to (9.27, -9.78), turned to 90 degrees
- moved R4 193.5 mm to (54.7, -39.0), turned to 0 degrees
- moved R1 188.6 mm to (11.2, -9.63), turned to 90 degrees
- moved U2 186.0 mm to (22.6, -5.33), turned to 90 degrees
- moved C2 183.8 mm to (7.37, -2.64)
- moved C1 183.1 mm to (7.37, -10.1)
- moved U1 179.5 mm to (10.2, -3.81), turned to 90 degrees
- moved D1 176.0 mm to (15.0, -10.0), turned to 0 degrees
- moved J2 173.3 mm to (2.80, -6.00), turned to -90 degrees
- moved C3 168.2 mm to (13.7, -4.57), turned to 0 degrees
- moved J3 164.4 mm to (33.2, -6.00), turned to -90 degrees
- moved C4 163.4 mm to (26.2, -7.62), turned to 0 degrees
Connections:
- C1 pad 1: +3V3 -> +5V
- C2 pad 1: Net-(C2-Pad1) -> +5V
- C3 pad 1: +5V -> +3V3
- C4 pad 1: +5V -> +3V3
- D1 pad 1: +5V -> GND
- D1 pad 2: GND -> Net-(D1-Pad2)
- D2 pad 1: GND -> +5V
- D2 pad 2: Net-(D2-Pad2) -> GND
- J1 pad 1: /COUNT -> +5V
- J1 pad 2: Net-(C2-Pad1) -> /SCLin
- J1 pad 3: GND -> /SDAin
- J2 pad 2: /SCL -> /SCLin
- J2 pad 3: /SDA -> /SDAin
- J3 pad 2: /SCL -> /SCLout
- J3 pad 3: /SDA -> /SDAout
- R1 pad 1: Net-(JP2-Pad2) -> +5V
- R1 pad 2: /COUNT -> Net-(D1-Pad2)
- R2 pad 1: Net-(C2-Pad1) -> +3V3
- R2 pad 2: Net-(JP2-Pad2) -> /SCLin
- R3 pad 2: /SDA -> /SDAin
- R4 pad 1: Net-(R4-Pad1) -> +3V3
- R4 pad 2: Net-(D2-Pad2) -> Net-(D3-Pad2)
- U1 pad 1: Net-(R4-Pad1) -> +5V
- U1 pad 2: (no net) -> GND
- U1 pad 3: Net-(JP1-Pad2) -> +5V
- U1 pad 4: GND -> (no net)
- U1 pad 5: /SDA -> +3V3
- U2 pad 1: (no net) -> +3V3
- U2 pad 2: /COUNT -> /SCLout
- U2 pad 3: GND -> /SCLin
- U2 pad 4: Net-(R4-Pad1) -> GND
- U2 pad 5: +3V3 -> Net-(D3-Pad2)
Routing:
- net /SCL: track 27.9 -> 0.00 mm
- net /SDA: track 25.6 -> 0.00 mm, vias 2 -> 0
- net /SDAin: track 0.00 -> 25.1 mm, vias 0 -> 1
- net /SCLin: track 0.00 -> 24.7 mm, vias 0 -> 3
- net +5V: track 45.8 -> 65.7 mm, vias 4 -> 2
- net +3V3: track 38.4 -> 19.3 mm, vias 3 -> 0
- net Net-(R4-Pad1): track 18.9 -> 0.00 mm
- net /SDAout: track 0.00 -> 17.9 mm, vias 0 -> 2
- net /SCLout: track 0.00 -> 14.1 mm, vias 0 -> 1
- net Net-(JP1-Pad2): track 13.9 -> 0.00 mm
- net /COUNT: track 12.6 -> 0.00 mm
- net Net-(JP2-Pad2): track 10.5 -> 0.00 mm
- net Net-(C2-Pad1): track 9.86 -> 0.00 mm
- net Net-(D2-Pad2): track 2.16 -> 0.00 mm
- net Net-(D1-Pad2): track 0.00 -> 1.92 mm
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- removed copper zone on B.Cu, net GND
- removed copper zone on F.Cu, net GND
Other:
- board size 37.5 x 19 mm -> 36 x 12 mm
- board text removed: "+5V"
- board text removed: "0X50"
- board text removed: "2021"
- board text removed: "GND"
- board text removed: "I2C"
- board text removed: "IN"
- board text removed: "PULSE"
- board text removed: "TFRPM01C"
- board text removed: "ThunderFly.cz"

Commit message: Edit PCB
Parts:
- added M2: M3, Mlab_Mechanical:dira_3mm, F.Cu at (22.6, -14.2)
- added M2: HOLE, Mlab_Mechanical:dira_3mm, F.Cu at (12.5, -15.0)
- added M3: HOLE, Mlab_Mechanical:dira_3mm, F.Cu at (2.50, 0.00)
- added M4: HOLE, Mlab_Mechanical:dira_3mm, F.Cu at (2.50, -15.0)
- added M5: HOLE, Mlab_Mechanical:dira_3mm, F.Cu at (22.5, -15.0)
- added M6: HOLE, Mlab_Mechanical:dira_3mm, F.Cu at (22.5, 0.00)
- M1: value M3 -> HOLE; footprint Mlab_Mechanical:MountingHole_3mm -> Mlab_Mechanical:dira_3mm
- moved M1 77.5 mm to (12.5, 0.00)
- moved R4 55.7 mm to (12.7, -2.54), turned to 180 degrees
- moved R2 55.1 mm to (15.2, -2.41), turned to 90 degrees
- moved R5 52.3 mm to (17.3, -2.41), turned to 90 degrees
- moved R3 48.3 mm to (15.2, -12.5), turned to -90 degrees
- moved R6 47.7 mm to (17.3, -12.5), turned to -90 degrees
- moved J3 11.1 mm to (22.2, -7.50)
- moved J4 11.1 mm to (22.2, -7.50)
- moved C4 8.69 mm to (17.7, -9.40), turned to 90 degrees
- moved U2 8.17 mm to (14.7, -7.50)
- moved D1 7.16 mm to (8.50, -13.0), turned to 180 degrees
- moved D3 6.50 mm to (8.50, -2.00), turned to 180 degrees
- moved C3 5.49 mm to (11.3, -9.50), turned to 90 degrees
- moved C2 4.68 mm to (11.2, -5.36)
- moved R1 3.44 mm to (12.7, -12.7), turned to 180 degrees
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Connections:
- U1 pad 4: (no net) -> unconnected-(U1-Pad4)
Routing:
- net GND: track 0.00 -> 21.6 mm, vias 0 -> 27
- net +5V: track 65.7 -> 48.6 mm, vias 2 -> 4
- net +3V3: track 19.3 -> 33.9 mm, vias 0 -> 2
- net Net-(D3-Pad2): track 0.00 -> 9.49 mm
- net /SCLin: track 24.7 -> 17.1 mm, vias 3 -> 2
- net /SDAin: track 25.1 -> 18.8 mm, vias 1 -> 2
- net /SDAout: track 17.9 -> 14.5 mm
- net /SCLout: track 14.1 -> 13.1 mm, vias 1 -> 2
- added copper zone on B.Cu, net GND
- added copper zone on F.Cu, net GND
Other:
- board size 36 x 12 mm -> 25 x 15 mm
- board text added: "TFI2CEXT01A"

Commit message: Layout improvement.
Routing:
- net GND: track 21.6 -> 23.4 mm

Commit message: Finishing the design
Routing:
- net GND: vias 27 -> 35
Other:
- board text added: "PWR"
- board text added: "READY"
Changed lines of the file:
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@@
-(kicad_pcb (version 20210228) (generator pcbnew)
+(kicad_pcb (version 20210126) (generator pcbnew)
   (general
     (thickness 1.6)
@@
       (dielectric_constraints no)
     )
-    (pad_to_mask_clearance 0)
     (aux_axis_origin 126.746 136.906)
     (grid_origin 126.746 136.906)
@@
     (pad "MP" smd roundrect (at -3.725 1.35 270) (locked) (size 1 2.7) (layers "F.Cu" "F.Paste" "F.Mask") (roundrect_rratio 0.25)
       (net 1 "GND") (pintype "input"))
-    (model "${KISYS3DMOD}/Connector_JST.3dshapes/JST_GH_SM04B-GHS-TB_1x04-1MP_P1.25mm_Horizontal.wrl"
+    (model "${KISYS3DMOD}/Connector_JST.3dshapes/JST_GH_SM04B-GHS-TB_1x04-1MP_P1.25mm_Horizontal.wrl" hide
       (offset (xyz 0 0 0))
       (scale (xyz 1 1 1))
@@
     (pad "MP" smd roundrect (at 3.725 1.35 90) (locked) (size 1 2.7) (layers "F.Cu" "F.Paste" "F.Mask") (roundrect_rratio 0.25)
       (net 1 "GND") (pintype "input"))
-    (model "${KISYS3DMOD}/Connector_JST.3dshapes/JST_GH_SM04B-GHS-TB_1x04-1MP_P1.25mm_Horizontal.wrl"
+    (model "${KISYS3DMOD}/Connector_JST.3dshapes/JST_GH_SM04B-GHS-TB_1x04-1MP_P1.25mm_Horizontal.wrl" hide
       (offset (xyz 0 0 0))
       (scale (xyz 1 1 1))
@@
     (pad "" np_thru_hole circle (at 0 0 180) (locked) (size 2.7 2.7) (drill 2.7) (layers *.Mask))
     (pad "1" smd rect (at 2.075 0 180) (locked) (size 0.95 1.5) (layers "B.Cu" "B.Paste" "B.Mask")
-      (net 1 "GND") (pinfunction "K") (pintype "passive"))
+      (net 1 "GND") (pinfunction "K"))
     (pad "2" smd rect (at -2.075 0 180) (locked) (size 0.95 1.5) (layers "B.Cu" "B.Paste" "B.Mask")
-      (net 4 "Net-(D1-Pad2)") (pinfunction "A") (pintype "passive"))
+      (net 4 "Net-(D1-Pad2)") (pinfunction "A"))
     (model "${KISYS3DMOD}/LED_SMD.3dshapes/LED_1206_3216Metric.wrl"
       (offset (xyz -0 0 0.5))
@@
   (gr_line (start 0 -15) (end 0 0) (layer "Edge.Cuts") (width 0.15) (locked))
   (gr_line (start 0 0) (end 25 0) (layer "Edge.Cuts") (width 0.15) (locked))
-  (gr_text "TFI2CEXT01A" (at 12.5 -5.207) (layer "F.SilkS")
+  (gr_text "PWR" (at 6.5 -10.5) (layer "F.SilkS")
+    (effects (font (size 1.3 1.3) (thickness 0.3)) (justify left))
+  )
+  (gr_text "READY" (at 6.5 -4.5) (layer "F.SilkS")
+    (effects (font (size 1.3 1.3) (thickness 0.3)) (justify left))
+  )
+  (gr_text "TFI2CEXT01A" (at 17.272 -7.5 90) (layer "F.SilkS")
     (effects (font (size 1.3 1.3) (thickness 0.3)))
   )
@@
     (pts (xy 25 0) (xy 25 -15))
     (height 2.621)
-    (gr_text "15 mm" (at 26.471 -7.5 90) (layer "Dwgs.User")
+    (gr_text "15 mm" (at 28.771 -7.5 90) (layer "Dwgs.User")
       (effects (font (size 1 1) (thickness 0.15)))
     )
@@
     (pts (xy 0 -15) (xy 2.5 -15))
     (height -2.119)
-    (gr_text "2,5 mm" (at 1.25 -18.269) (layer "Dwgs.User")
+    (gr_text "2.5 mm" (at 1.25 -18.269) (layer "Dwgs.User")
       (effects (font (size 1 1) (thickness 0.15)))
     )
@@
     (pts (xy 0 0) (xy 25 0))
     (height 4.881)
-    (gr_text "25 mm" (at 12.5 3.731) (layer "Dwgs.User")
+    (gr_text "25 mm" (at 12.5 6.031) (layer "Dwgs.User")
       (effects (font (size 1 1) (thickness 0.15)))
     )
@@
   (segment (start 1.256371 -7.860371) (end 1.016 -7.62) (width 0.4) (layer "F.Cu") (net 1))
   (segment (start 1.256371 -9.210907) (end 1.256371 -7.860371) (width 0.4) (layer "F.Cu") (net 1))
+  (via (at 23.114 -2.032) (size 0.8) (drill 0.4) (layers "F.Cu" "B.Cu") (free) (net 1))
+  (via (at 3.048 -2.032) (size 0.8) (drill 0.4) (layers "F.Cu" "B.Cu") (free) (net 1))
+  (via (at 23.114 -12.954) (size 0.8) (drill 0.4) (layers "F.Cu" "B.Cu") (free) (net 1))
   (via (at 20.955 -2.667) (size 0.8) (drill 0.4) (layers "F.Cu" "B.Cu") (free) (net 1))
+  (via (at 3.048 -12.954) (size 0.8) (drill 0.4) (layers "F.Cu" "B.Cu") (free) (net 1))
   (via (at 4.445 -1.905) (size 0.8) (drill 0.4) (layers "F.Cu" "B.Cu") (free) (net 1))
   (via (at 6.223 -4.318) (size 0.8) (drill 0.4) (layers "F.Cu" "B.Cu") (net 1))
@@
   (via (at 20.32 -12.573) (size 0.8) (drill 0.4) (layers "F.Cu" "B.Cu") (free) (net 1))
   (via (at 8.226998 -8.509) (size 0.8) (drill 0.4) (layers "F.Cu" "B.Cu") (net 1))
+  (via (at 1.016 -2.032) (size 0.8) (drill 0.4) (layers "F.Cu" "B.Cu") (free) (net 1))
   (via (at 4.064 -12.827) (size 0.8) (drill 0.4) (layers "F.Cu" "B.Cu") (free) (net 1))
   (via (at 19.685 -1.397) (size 0.8) (drill 0.4) (layers "F.Cu" "B.Cu") (free) (net 1))
   (via (at 4.572 -3.81) (size 0.8) (drill 0.4) (layers "F.Cu" "B.Cu") (free) (net 1))
+  (via (at 1.016 -12.954) (size 0.8) (drill 0.4) (layers "F.Cu" "B.Cu") (free) (net 1))
   (via (at 24.003 -5.588) (size 0.8) (drill 0.4) (layers "F.Cu" "B.Cu") (free) (net 1))
   (via (at 20.955 -4.064) (size 0.8) (drill 0.4) (layers "F.Cu" "B.Cu") (free) (net 1))
+  (via (at 24.13 -12.954) (size 0.8) (drill 0.4) (layers "F.Cu" "B.Cu") (free) (net 1))
+  (via (at 24.13 -2.032) (size 0.8) (drill 0.4) (layers "F.Cu" "B.Cu") (free) (net 1))
   (via (at 1.016 -7.62) (size 0.8) (drill 0.4) (layers "F.Cu" "B.Cu") (net 1))
   (via (at 21.463 -12.954) (size 0.8) (drill 0.4) (layers "F.Cu" "B.Cu") (free) (net 1))
