File: hw/sch_pcb/TFI2CEXT01.kicad_pcb (KiCad board)
At the start: 2 copper layers, 25 x 15 mm, 26 parts, among them J1 SM04B-GHS-TB, J2 SM04B-GHS-TB, J3 SM04B-GHS-TB, J4 SM04B-GHS-TB, M1 HOLE, M2 HOLE, M2 M3, M3 HOLE, M4 HOLE, M5 HOLE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

Commit message: Upravy pred vyrobou 01B
Parts:
- removed the M2 at (22.6, -14.2)
- added G1: LOGO, MLAB_LOGA:TF 10x4,7, F.Cu at (11.9, -6.10)
- C1: footprint Mlab_R:SMD-0805 -> Capacitor_SMD:C_0805_2012Metric
- C2, C3, C4, R2, R3, R5, R6: footprint Mlab_R:SMD-0603 -> Resistor_SMD:R_0603_1608Metric
- D1, D3: footprint Mlab_D:LED_1206 -> Mlab_D:LED_1206_mill
- R1: value 180R -> 130R; footprint Mlab_R:SMD-0603 -> Resistor_SMD:R_0603_1608Metric
- R4: value 180R -> 287R; footprint Mlab_R:SMD-0603 -> Resistor_SMD:R_0603_1608Metric
Routing:
- net Net-(D3-A): track 9.49 -> 11.3 mm
- net GND: vias 35 -> 33
Other:
- board text added: "TFI2CEXT01B"
- board text removed: "TFI2CEXT01A"
