File: hw/sch_pcb/TFI2CEXT01.kicad_sch (KiCad schematic)
At the start: 25 parts, among them J1 SM04B-GHS-TB, J2 SM04B-GHS-TB, J3 SM04B-GHS-TB, J4 SM04B-GHS-TB, M1 HOLE, M2 HOLE, M3 HOLE, M4 HOLE, M5 HOLE, M6 HOLE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

Commit message: Upravy pred vyrobou 01B
Parts:
- added G1: LOGO, MLAB_LOGA:TF 10x4,7, symbol MLAB_TF_LOGO:LOGO
- C1: footprint Mlab_R:SMD-0805 -> Capacitor_SMD:C_0805_2012Metric
- C2, C3, C4, R2, R3, R5, R6: footprint Mlab_R:SMD-0603 -> Resistor_SMD:R_0603_1608Metric
- D1, D3: footprint Mlab_D:LED_1206 -> Mlab_D:LED_1206_mill
- R1: value 180R -> 130R; footprint Mlab_R:SMD-0603 -> Resistor_SMD:R_0603_1608Metric; UST_ID 5c70984512875079b91f8957 -> (none)
- R4: value 180R -> 287R; footprint Mlab_R:SMD-0603 -> Resistor_SMD:R_0603_1608Metric; UST_ID 5c70984512875079b91f8957 -> (none)

Commit message: Edit UST_ID
Parts:
- R1: UST_ID (none) -> 5cd08b17128750448e4542b1
- R4: UST_ID (none) -> 651a975c462c6d9e7205504d
Changed lines of the file:
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@@
       (effects (font (size 1.27 1.27)) hide)
     )
-    (property "UST_ID" "" (at 140.97 87.63 0)
+    (property "UST_ID" "651a975c462c6d9e7205504d" (at 140.97 87.63 0)
       (effects (font (size 1.27 1.27)) hide)
     )
@@
       (effects (font (size 1.27 1.27)) hide)
     )
-    (property "UST_ID" "" (at 19.05 168.91 0)
-      (effects (font (size 1.27 1.27)) hide)
-    )
+    (property "UST_ID" "5cd08b17128750448e4542b1" (at 19.05 168.91 0)
+      (effects (font (size 1.27 1.27)) hide)
+    )
